File: CAD/coffee_grams.kicad_pcb (KiCad board)
At the start: 2 copper layers, 46 parts, among them J1 USB_B_Mini, J3 Conn_01x05_Male, Q1 MMBT4403, Q2 BC847, Q3 BC847, SW1 BX_TARE, SW2 BX_ON_OFF, SW3 BX_TIMER, SW4 BX_COFFEE_G, SW5 BX_H2O_G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

Commit message: completed 0.1 board
Parts:
- removed C13: .1u, Capacitor_SMD:C_0805_2012Metric_Pad1.15x1.40mm_HandSolder
- removed C14: 10u, Capacitor_SMD:C_0805_2012Metric_Pad1.15x1.40mm_HandSolder
- removed C15: 33u, Capacitor_SMD:C_0805_2012Metric_Pad1.15x1.40mm_HandSolder
- removed J3: Conn_01x05_Male, Connector_PinSocket_2.54mm:PinSocket_1x05_P2.54mm_Vertical
- added J2: Conn_01x05_Male, Connector_PinSocket_2.54mm:PinSocket_1x05_P2.54mm_Vertical, F.Cu at (109.5, 61.0)
- C1: value 0.1u -> 4.7n
- C11: value 4.7n -> 10u
- C12: value .47u -> 33u
- C2: value 10u -> .1u
- C3, C6: value 0.1u -> 10u
- C4: value 0.1u -> .1u
- C5: value 10u -> 0.1u
- C8: value .1u -> 0.1u
- C9: value 10u -> .47u
- Q1: value MMBT4403 -> BC847
- Q3: value BC847 -> MMBT4403
- R1: value 20k -> 1M
- R2: value 8.2k -> 12K
- R3: value 100 -> 12K
- R4: value 100 -> 20k
- R5: value 10k -> 8.2k
- R6: value 1M -> 100
- R7: value 12K -> 100
- R8: value 12K -> 10k
- U1: value HX711 -> FT232RL; footprint Package_SO:SOP-16_4.4x10.4mm_P1.27mm -> Package_SO:SSOP-28_5.3x10.2mm_P0.65mm
- U2: value FT232RL -> HX711; footprint Package_SO:SSOP-28_5.3x10.2mm_P0.65mm -> Package_SO:SOP-16_4.4x10.4mm_P1.27mm
- moved RV1 85.0 mm to (136.2, 100.4), turned to 0 degrees
- moved U3 82.4 mm to (156.6, 85.5), turned to 270 degrees
- moved C3 71.9 mm to (137.0, 77.0), turned to 0 degrees
- moved R11 67.6 mm to (163.0, 101.0), turned to 270 degrees
- moved R9 61.7 mm to (158.0, 101.0), turned to 90 degrees
- moved C8 55.4 mm to (108.0, 67.0), turned to 180 degrees
- moved C11 50.0 mm to (131.0, 72.0)
- moved R10 48.3 mm to (152.0, 101.0), turned to 90 degrees
- moved R12 47.1 mm to (146.8, 101.0), turned to 270 degrees
- moved R1 46.6 mm to (101.0, 84.0), turned to 180 degrees
- moved Q3 45.3 mm to (154.0, 69.0), turned to 270 degrees
- moved C2 44.4 mm to (131.0, 77.0)
- moved U4 40.9 mm to (115.8, 74.0), turned to 180 degrees
- moved Q2 39.4 mm to (138.0, 83.0), turned to 0 degrees
- moved U1 39.2 mm to (117.4, 90.8), turned to 180 degrees
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Connections:
- C1 pad 1: +5V -> Net-(C1-Pad1)
- C10 pad 1: Net-(C10-Pad1) -> +3V3
- C11 pad 1: Net-(C11-Pad1) -> +3V3
- C12 pad 1: +5V -> +3V3
- C3 pad 1: +3V3 -> +5V
- C4 pad 1: /AVDD -> Net-(C4-Pad1)
- C6 pad 1: Net-(C6-Pad1) -> /AVDD
- C7 pad 1: /INPA -> Net-(C7-Pad1)
- C7 pad 2: /INNA -> GND
- C8 pad 1: +5V -> /INPA
- C8 pad 2: GND -> /INNA
- J1 pad 6: Net-(C11-Pad1) -> Net-(C1-Pad1)
- Q1 pad 2: Net-(L1-Pad2) -> /DTR
- Q1 pad 3: +5V -> /IO0
- Q2 pad 2: /DTR -> /RTS
- Q2 pad 3: /IO0 -> /EN
- Q3 pad 2: /RTS -> Net-(L1-Pad2)
- Q3 pad 3: /EN -> +5V
- R1 pad 1: Net-(L1-Pad2) -> Net-(C1-Pad1)
- R1 pad 2: Net-(R1-Pad2) -> GND
- R2 pad 1: GND -> Net-(Q1-Pad1)
- R2 pad 2: Net-(R1-Pad2) -> /RTS
- R3 pad 1: /INNA -> Net-(Q2-Pad1)
- R3 pad 2: /A- -> /DTR
- R4 pad 1: /INPA -> Net-(L1-Pad2)
- R4 pad 2: /A+ -> Net-(R4-Pad2)
- R5 pad 1: +5V -> GND
- R5 pad 2: Net-(JP1-Pad1) -> Net-(R4-Pad2)
- R6 pad 1: Net-(C11-Pad1) -> /INNA
- R6 pad 2: GND -> /A-
- R7 pad 1: Net-(Q2-Pad1) -> /INPA
- R7 pad 2: /RTS -> /A+
- R8 pad 1: Net-(Q3-Pad1) -> +5V
- R8 pad 2: /DTR -> Net-(JP1-Pad1)
- U1 pad 1: +5V -> /RXD0
- U1 pad 11: /HX_SCK -> Net-(U1-Pad11)
- U1 pad 12: /HX_DOUT -> Net-(U1-Pad12)
- U1 pad 14: GND -> Net-(U1-Pad14)
- U1 pad 15: Net-(JP1-Pad1) -> Net-(J1-Pad3)
- U1 pad 16: +3V3 -> Net-(J1-Pad2)
- U1 pad 2: Net-(Q1-Pad1) -> /DTR
- U1 pad 3: Net-(L1-Pad2) -> /RTS
- U1 pad 4: Net-(R1-Pad2) -> Net-(C4-Pad1)
- U1 pad 5: GND -> /TXD0
- U1 pad 6: Net-(C6-Pad1) -> Net-(U1-Pad6)
- U1 pad 7: /INNA -> GND
- U1 pad 8: /INPA -> (no net)
- U2 pad 1: /RXD0 -> +5V
- U2 pad 11: Net-(U2-Pad11) -> /HX_SCK
- U2 pad 12: Net-(U2-Pad12) -> /HX_DOUT
- U2 pad 14: Net-(U2-Pad14) -> GND
- U2 pad 15: Net-(J1-Pad3) -> Net-(JP1-Pad1)
- U2 pad 16: Net-(J1-Pad2) -> +3V3
- U2 pad 2: /DTR -> Net-(Q3-Pad1)
- U2 pad 3: /RTS -> Net-(L1-Pad2)
- U2 pad 4: Net-(C10-Pad1) -> Net-(R4-Pad2)
- U2 pad 5: /TXD0 -> GND
- U2 pad 6: Net-(U2-Pad6) -> Net-(C7-Pad1)
- U2 pad 7: GND -> /INNA
- U2 pad 8: (no net) -> /INPA
- U3 pad 11: /BX_COFFEE_G -> /BX_TARE
- U3 pad 12: /BX_H2O_G -> /BX_ON_OFF
- U3 pad 23: /LCD_D7 -> /LCD_D0
- U3 pad 24: /LCD_D6 -> /LCD_D1
- U3 pad 26: /LCD_D5 -> /LCD_D2
- U3 pad 27: /LCD_D4 -> /LCD_D3
- U3 pad 28: /LCD_D3 -> /LCD_D4
- U3 pad 29: /LCD_D2 -> /LCD_D5
- U3 pad 30: /LCD_D1 -> /LCD_D6
- U3 pad 31: /LCD_D0 -> /LCD_D7
- U3 pad 8: /BX_ON_OFF -> /BX_H2O_G
- U3 pad 9: /BX_TARE -> /BX_COFFEE_G
Routing:
- net +5V: track 0.00 -> 159.9 mm, vias 0 -> 4
- net /BX_ON_OFF: track 0.00 -> 108.6 mm, vias 0 -> 1
- net /BX_TARE: track 0.00 -> 97.7 mm, vias 0 -> 1
- net /BX_H2O_G: track 0.00 -> 88.8 mm, vias 0 -> 1
- net /BX_TIMER: track 0.00 -> 86.6 mm, vias 0 -> 1
- net GND: track 0.00 -> 85.4 mm, vias 0 -> 13
- net /BX_COFFEE_G: track 0.00 -> 82.5 mm, vias 0 -> 1
- net /LCD_RS: track 0.00 -> 76.9 mm, vias 0 -> 2
- net /LCD_E: track 0.00 -> 68.6 mm, vias 0 -> 2
- net +3V3: track 0.00 -> 62.1 mm, vias 0 -> 2
- net Net-(DS1-Pad15): track 0.00 -> 55.7 mm, vias 0 -> 3
- net /HX_DOUT: track 0.00 -> 47.8 mm, vias 0 -> 2
- net /LCD_D0: track 0.00 -> 47.8 mm, vias 0 -> 1
- net /TXD0: track 0.00 -> 47.5 mm, vias 0 -> 2
- net /LCD_D1: track 0.00 -> 46.5 mm, vias 0 -> 1
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- added copper zone on B.Cu, net GND
- added copper zone on F.Cu, net GND
Other:
- board outline added: 81 x 99 mm
- board text added: "Coffee Grams Enoch Chau 2020"
