File: CAD/coffee_grams.sch (KiCad schematic (older format))
At the start: 11 parts, among them J1 Conn_01x05_Male, SW1 SW_Push_Dual, SW2 SW_Push_Dual, SW3 SW_Push_Dual, SW4 SW_Push_Dual, SW5 SW_Push_Dual, U1 HX711

Commit message: completed schematic, started pcb
Parts:
- removed C1, C3: 0.1u, symbol Device:C
- removed C2: 10u, symbol Device:C
- removed J1, J?: Conn_01x05_Male, symbol Connector:Conn_01x05_Male
- added C10, C13, C8: .1u, Capacitor_SMD:C_0805_2012Metric_Pad1.15x1.40mm_HandSolder, symbol Device:C
- added C11: 4.7n, Capacitor_SMD:C_0805_2012Metric_Pad1.15x1.40mm_HandSolder, symbol Device:C
- added C12: .47u, Capacitor_SMD:C_0805_2012Metric_Pad1.15x1.40mm_HandSolder, symbol Device:C
- added C14, C5, C9: 10u, Capacitor_SMD:C_0805_2012Metric_Pad1.15x1.40mm_HandSolder, symbol Device:C
- added C15: 33u, Capacitor_SMD:C_0805_2012Metric_Pad1.15x1.40mm_HandSolder, symbol Device:C
- added C4, C6, C7: 0.1u, Capacitor_SMD:C_0805_2012Metric_Pad1.15x1.40mm_HandSolder, symbol Device:C
- added DS1: WC1602A, Display:WC1602A, symbol Display_Character:WC1602A
- added J1: USB_B_Mini, Connector_USB:USB_Mini-B_Wuerth_65100516121_Horizontal, symbol Connector:USB_B_Mini
- added J3: Conn_01x05_Male, Connector_PinSocket_2.54mm:PinSocket_1x05_P2.54mm_Vertical, symbol Connector:Conn_01x05_Male
- added JP1: Jumper, Jumper:SolderJumper-2_P1.3mm_Open_Pad1.0x1.5mm, symbol Device:Jumper
- added L1: 3.3u, Inductor_SMD:L_0805_2012Metric_Pad1.15x1.40mm_HandSolder, symbol Device:L
- added Q1: MMBT4403, Package_TO_SOT_SMD:SOT-23, symbol Device:Q_PNP_BCE
- added Q2, Q3: BC847, Package_TO_SOT_SMD:SOT-23, symbol Transistor_BJT:BC847
- added R1: 20k, Resistor_SMD:R_0805_2012Metric_Pad1.15x1.40mm_HandSolder, symbol Device:R
- added R10, R9: 150, Resistor_SMD:R_0805_2012Metric_Pad1.15x1.40mm_HandSolder, symbol Device:R
- added R11: 4.7k, Resistor_SMD:R_0805_2012Metric_Pad1.15x1.40mm_HandSolder, symbol Device:R
- added R12: 4.7K, Resistor_SMD:R_0805_2012Metric_Pad1.15x1.40mm_HandSolder, symbol Device:R
- added R13: 220, Resistor_SMD:R_0805_2012Metric_Pad1.15x1.40mm_HandSolder, symbol Device:R
- added R2: 8.2k, Resistor_SMD:R_0805_2012Metric_Pad1.15x1.40mm_HandSolder, symbol Device:R
- added R3, R4: 100, Resistor_SMD:R_0805_2012Metric_Pad1.15x1.40mm_HandSolder, symbol Device:R
- added R5: 10k, Resistor_SMD:R_0805_2012Metric_Pad1.15x1.40mm_HandSolder, symbol Device:R
- added R6: 1M, Resistor_SMD:R_0805_2012Metric_Pad1.15x1.40mm_HandSolder, symbol Device:R
- added R7, R8: 12K, Resistor_SMD:R_0805_2012Metric_Pad1.15x1.40mm_HandSolder, symbol Device:R
- added RV1: 10K, Potentiometer_THT:Potentiometer_Bourns_3266W_Vertical, symbol Device:R_POT
- added U2: FT232RL, Package_SO:SSOP-28_5.3x10.2mm_P0.65mm, symbol Interface_USB:FT232RL
- added U3: ESP32-WROOM-32, RF_Module:ESP32-WROOM-32, symbol RF_Module:ESP32-WROOM-32
- added U4: LM3940, Package_TO_SOT_SMD:SOT-223, symbol coffee_grams:LM3940
- SW1: value SW_Push_Dual -> BX_TARE; footprint (none) -> Button_Switch_THT:SW_TH_Tactile_Omron_B3F-10xx
- SW2: value SW_Push_Dual -> BX_ON_OFF; footprint (none) -> Button_Switch_THT:SW_TH_Tactile_Omron_B3F-10xx
- SW3: value SW_Push_Dual -> BX_TIMER; footprint (none) -> Button_Switch_THT:SW_TH_Tactile_Omron_B3F-10xx
- SW4: value SW_Push_Dual -> BX_COFFEE_G; footprint (none) -> Button_Switch_THT:SW_TH_Tactile_Omron_B3F-10xx
- SW5: value SW_Push_Dual -> BX_H2O_G; footprint (none) -> Button_Switch_THT:SW_TH_Tactile_Omron_B3F-10xx
- U1: footprint (none) -> Package_SO:SOP-16_4.4x10.4mm_P1.27mm
Connections:
- net GND: now also SW1.1, SW1.3, SW2.1, SW2.3, SW3.1, SW3.3, SW4.1, SW4.3, SW5.1, SW5.3, U1.14 (XI), U1.5 (AGND), C10.2, C11.2, C12.2, C13.2, C14.2, C15.2, C4.2, C5.2, C6.2, C8.2, C9.2, DS1.1 (VSS), DS1.16 (LED(-)), DS1.5 (R/W), J1.5 (GND), J3.2 (Pin_2), J3.5 (Pin_5), JP1.2, R11.1, R12.1, R2.1, R6.2, RV1.1, U2.18 (GND), U2.21 (GND), U2.25 (AGND), U2.26 (TEST), U2.7 (GND), U3.1 (GND), U3.15 (GND), U3.38 (GND), U3.39 (GND), U4.2 (GND), U4.4 (GND)
- net BX_ON_OFF: now reaches SW2.2
- net BX_ON_OFF: now also SW2.4, U3.8 (IO32)
- net BX_TARE: now reaches SW1.2
- net BX_TARE: now also SW1.4, U3.9 (IO33)
- net BX_TIMER: now reaches SW3.2
- net BX_TIMER: now also SW3.4, U3.10 (IO25)
- net BX_H2O_G: now reaches SW5.2
- net BX_H2O_G: now also SW5.4, U3.12 (IO27)
- net BX_COFFEE_G: now reaches SW4.2
- net BX_COFFEE_G: now also SW4.4, U3.11 (IO26)
- net HX_SCK: now reaches U1.11 (PC_SCK)
- net HX_SCK: now also U3.6 (IO34)
- net HX_DOUT: now reaches U1.12 (DOUT)
- net HX_DOUT: now also U3.7 (IO35)
- net at U1.15 (RATE): now also JP1.1, R5.2
- net at U1.2 (BASE): now also Q1.1 (B)
- net at U1.3 (AVDD): now also L1.2, Q1.2 (C), R1.1
- net at U1.4 (VFB): now also R1.2, R2.2
- net at U1.6 (VBG): now also C6.1
- net INNA: now reaches U1.7 (INNA)
- net INNA: now also C7.2, R3.1
- net INPA: now reaches U1.8 (INPA)
- net INPA: now also C7.1, R4.1
- net VCC renamed +5V
- net +5V: now also C12.1, C8.1, C9.1, DS1.2 (VDD), J1.1 (VBUS), Q1.3 (E), R13.1, R5.1, RV1.3, U2.20 (VCC), U4.1 (IN)
- net VDD renamed +3V3
- net +3V3: now also C13.1, C14.1, C15.1, U3.2 (VDD), U4.3 (OUT)
- new net: J1.3 (D+), U2.15 (USBD+)
- new net: J1.2 (D-), U2.16 (USBD-)
- new net: C10.1, U2.17 (3V3OUT), U2.4 (VCCIO)
- new net: C11.1, J1.6 (Shield), R6.1
- new net: R9.2, U3.35 (TXD0/IO1)
- new net: R10.2, U3.34 (RXD0/IO3)
- new net: Q3.1 (B), R8.1
- new net: Q2.1 (B), R7.1
- new net: DS1.15 (LED(+)), R13.2
- new net: DS1.3 (VO), RV1.2
- new net A+: J3.4 (Pin_4), R4.2
- new net A-: J3.3 (Pin_3), R3.2
- new net AVDD: C4.1, C5.1, J3.1 (Pin_1), L1.1
- new net DTR: Q2.2 (E), R8.2, U2.2 (DTR)
- new net EN: Q3.3 (C), U3.3 (EN)
- new net IO0: Q2.3 (C), U3.25 (IO0)
- new net LCD_D0: DS1.7 (D0), U3.31 (IO19)
- new net LCD_D1: DS1.8 (D1), U3.30 (IO18)
- new net LCD_D2: DS1.9 (D2), U3.29 (IO5)
- new net LCD_D3: DS1.10 (D3), U3.28 (IO17)
- new net LCD_D4: DS1.11 (D4), U3.27 (IO16)
- new net LCD_D5: DS1.12 (D5), U3.26 (IO4)
- new net LCD_D6: DS1.13 (D6), U3.24 (IO2)
- new net LCD_D7: DS1.14 (D7), U3.23 (IO15)
- new net LCD_E: DS1.6 (E), U3.33 (IO21)
- new net LCD_RS: DS1.4 (RS), U3.37 (IO23)
- new net RTS: Q3.2 (E), R7.2, U2.3 (RTS)
- new net RXD0: R10.1, R12.2, U2.1 (TXD)
- new net TXD0: R11.2, R9.1, U2.5 (RXD)
- no-connect marks 0 -> 28
Other:
- note added: "16x2 LCD"
- note added: "5V to 3.3V"
- note added: "A+"
- note added: "A-"
- note added: "AVDD=VBG(R1+R2)/R2"
- note added: "Default: Closed - Data rate: 10 SPS\nOpen - 80 SPS, more noise per read"
- note added: "E+"
- note added: "E-"
- note added: "ESP32"
- note added: "FTDI Chip"
- note added: "HX711 Load Cell Amplifier\n"
- note added: "Shield"
- note added: "Tactile Switches"
- moved on the sheet: SW1, SW2, SW3, SW4, SW5, U1

Commit message: completed 0.1 board
Parts:
- renumbered C11 to C1, C13 to C10, C14 to C11, C15 to C12, C8 to C2, C9 to C3, C10 to C4, C4 to C5, C5 to C6, C6 to C7, C7 to C8, C12 to C9, J3 to J2, Q2 to Q1, Q3 to Q2, Q1 to Q3, R6 to R1, R7 to R2, R8 to R3, R1 to R4, R2 to R5, R3 to R6, R4 to R7, R5 to R8, U2 to U1, U1 to U2
Connections:
- net BX_COFFEE_G: now also U3.9 (IO33); no longer U3.11 (IO26)
- net BX_H2O_G: now also U3.8 (IO32); no longer U3.12 (IO27)
- net BX_ON_OFF: now also U3.12 (IO27); no longer U3.8 (IO32)
- net BX_TARE: now also U3.11 (IO26); no longer U3.9 (IO33)
- net LCD_D0: now also U3.23 (IO15); no longer U3.31 (IO19)
- net LCD_D1: now also U3.24 (IO2); no longer U3.30 (IO18)
- net LCD_D2: now also U3.26 (IO4); no longer U3.29 (IO5)
- net LCD_D3: now also U3.27 (IO16); no longer U3.28 (IO17)
- net LCD_D4: now also U3.28 (IO17); no longer U3.27 (IO16)
- net LCD_D5: now also U3.29 (IO5); no longer U3.26 (IO4)
- net LCD_D6: now also U3.30 (IO18); no longer U3.24 (IO2)
- net LCD_D7: now also U3.31 (IO19); no longer U3.23 (IO15)
