File: CAD/esp32/coffee_grams.sch (KiCad schematic (older format))
At the start: 43 parts, among them J1 USB_B_Mini, J2 Conn_01x05_Male, Q1 BC847, Q2 BC847, Q3 MMBT4403, SW1 BX_TARE, SW2 BX_ON_OFF, SW3 BX_TIMER, SW4 BX_COFFEE_G, SW5 BX_H2O_G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

Commit message: create r-pi pcb files
Parts:
- added C13, C15: .1u, Capacitor_SMD:C_0805_2012Metric_Pad1.15x1.40mm_HandSolder, symbol Device:C
- added C14: 10u, Capacitor_SMD:C_0805_2012Metric_Pad1.15x1.40mm_HandSolder, symbol Device:C
Connections:
- net +3V3: now also C15.1
- net +5V: now also C13.1, C14.1
- net GND: now also C13.2, C14.2, C15.2
Changed lines of the file:
@@
 encoding utf-8
 Sheet 1 1
-Title ""
-Date ""
-Rev ""
-Comp ""
+Title "Coffee Grams"
+Date "2020-05-19"
+Rev "0.1"
+Comp "Enoch Chau"
 Comment1 ""
 Comment2 ""
@@
 	2450 6250 2450 7100
 Connection ~ 2450 7100
+$Comp
+L Device:C C13
+U 1 1 5EC60002
+P 7350 1500
+F 0 "C13" H 7465 1546 50  0000 L CNN
+F 1 ".1u" H 7465 1455 50  0000 L CNN
+F 2 "Capacitor_SMD:C_0805_2012Metric_Pad1.15x1.40mm_HandSolder" H 7388 1350 50  0001 C CNN
+F 3 "~" H 7350 1500 50  0001 C CNN
+	1    7350 1500
+	1    0    0    -1
+$EndComp
+$Comp
+L Device:C C14
+U 1 1 5EC607C9
+P 7700 1500
+F 0 "C14" H 7815 1546 50  0000 L CNN
+F 1 "10u" H 7815 1455 50  0000 L CNN
+F 2 "Capacitor_SMD:C_0805_2012Metric_Pad1.15x1.40mm_HandSolder" H 7738 1350 50  0001 C CNN
+F 3 "~" H 7700 1500 50  0001 C CNN
+	1    7700 1500
+	1    0    0    -1
+$EndComp
+Wire Wire Line
+	7350 1350 7700 1350
+Wire Wire Line
+	8550 1400 8550 1350
+Connection ~ 8550 1350
+Wire Wire Line
+	7350 1650 7350 1800
+Wire Wire Line
+	7700 1650 7700 1800
+$Comp
+L power:GND #PWR037
+U 1 1 5EC8E12D
+P 7350 1800
+F 0 "#PWR037" H 7350 1550 50  0001 C CNN
+F 1 "GND" H 7355 1627 50  0000 C CNN
+F 2 "" H 7350 1800 50  0001 C CNN
+F 3 "" H 7350 1800 50  0001 C CNN
+	1    7350 1800
+	1    0    0    -1
+$EndComp
+$Comp
+L power:GND #PWR038
+U 1 1 5EC8E594
+P 7700 1800
+F 0 "#PWR038" H 7700 1550 50  0001 C CNN
+F 1 "GND" H 7705 1627 50  0000 C CNN
+F 2 "" H 7700 1800 50  0001 C CNN
+F 3 "" H 7700 1800 50  0001 C CNN
+	1    7700 1800
+	1    0    0    -1
+$EndComp
+Wire Wire Line
+	7100 1350 7350 1350
+Connection ~ 7100 1350
+Connection ~ 7350 1350
+$Comp
+L Device:C C15
+U 1 1 5ECAF563
+P 8550 1550
+F 0 "C15" H 8665 1596 50  0000 L CNN
+F 1 ".1u" H 8665 1505 50  0000 L CNN
+F 2 "Capacitor_SMD:C_0805_2012Metric_Pad1.15x1.40mm_HandSolder" H 8588 1400 50  0001 C CNN
+F 3 "~" H 8550 1550 50  0001 C CNN
+	1    8550 1550
+	1    0    0    -1
+$EndComp
+$Comp
+L power:GND #PWR0101
+U 1 1 5ECAF9C1
+P 8550 1850
+F 0 "#PWR0101" H 8550 1600 50  0001 C CNN
+F 1 "GND" H 8555 1677 50  0000 C CNN
+F 2 "" H 8550 1850 50  0001 C CNN
+F 3 "" H 8550 1850 50  0001 C CNN
+	1    8550 1850
+	1    0    0    -1
+$EndComp
+Wire Wire Line
+	8550 1700 8550 1850
 $EndSCHEMATC

Commit message: pcb rev2
Parts:
- J1: symbol Connector:USB_B_Mini -> coffee_grams-rescue:USB_B_Mini-Connector
Connections:
- net BX_ON_OFF: now also U3.37 (IO23); no longer U3.12 (IO27)
- net BX_TARE: now also U3.36 (IO22); no longer U3.11 (IO26)
- net LCD_E: now also U3.16 (IO13); no longer U3.33 (IO21)
- net LCD_RS: now also U3.13 (IO14); no longer U3.37 (IO23)
Changed lines of the file:
@@
 	1800 7650 1800 7100
 $Comp
-L Connector:USB_B_Mini J1
+L coffee_grams-rescue:USB_B_Mini-Connector J1
 U 1 1 5EDB6F28
 P 1500 7850
@@
 Text Label 12600 8200 0    50   ~ 0
 LCD_D7
-Wire Wire Line
-	8800 8150 9200 8150
-Text Label 9200 8350 0    50   ~ 0
+Text Label 9200 7550 0    50   ~ 0
 LCD_RS
-Text Label 9200 8150 0    50   ~ 0
-LCD_E
 $Comp
 L RF_Module:ESP32-WROOM-32 U3
@@
 	8800 9050 9250 9050
 Wire Wire Line
-	8800 8350 9200 8350
+	8800 7550 9200 7550
 Wire Wire Line
 	8800 8050 9200 8050
-Text Label 9200 7650 0    50   ~ 0
-LCD_D0
 Text Label 9200 6950 0    50   ~ 0
 LCD_D1
@@
 LCD_D7
 Wire Wire Line
-	8800 7650 9200 7650
-Wire Wire Line
 	8800 8850 9250 8850
 Wire Wire Line
 	8800 8750 9250 8750
-Text Label 9200 8550 0    50   ~ 0
+Text Label 9200 8250 0    50   ~ 0
 BX_TARE
-Text Label 9200 8650 0    50   ~ 0
-BX_ON_OFF
 Wire Wire Line
 	8800 8450 9200 8450
@@
 BX_TIMER
 Wire Wire Line
-	8800 8550 9200 8550
-Wire Wire Line
-	8800 8650 9200 8650
+	8800 8250 9200 8250
 Text Label 9250 8850 0    50   ~ 0
 BX_COFFEE_G
-Text Label 9250 8750 0    50   ~ 0
-BX_H2O_G
 NoConn ~ 8800 7350
-NoConn ~ 8800 7450
-NoConn ~ 8800 7550
 Wire Wire Line
 	8200 6550 8200 6000
@@
 Wire Wire Line
 	13650 6800 13650 6300
-NoConn ~ 8800 8250
+NoConn ~ 8800 8550
 $Comp
 L power:+3.3V #PWR015
@@
 Wire Wire Line
 	8550 1700 8550 1850
+Wire Wire Line
+	8800 7650 9200 7650
+NoConn ~ 8800 8150
+NoConn ~ 8800 8650
+Text Label 9200 7650 0    50   ~ 0
+LCD_D0
+Wire Wire Line
+	8800 7450 9200 7450
+Text Label 9200 7450 0    50   ~ 0
+LCD_E
+Text Label 9250 8750 0    50   ~ 0
+BX_H2O_G
+Wire Wire Line
+	8800 8350 9200 8350
+Text Label 9200 8350 0    50   ~ 0
+BX_ON_OFF
 $EndSCHEMATC
